File: OpenC16Cart.sch (KiCad schematic (older format))
At the start: 15 parts, among them J1 CONN_02X03, J11 CONN_01X03, J12 CONN_01X03, J2 CONN_01X03, J21 CONN_01X03, J22 CONN_01X03, J3 CONN_01X03, J4 CONN_02X03, J5 CONN_01X03, J6 CONN_01X03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

Commit message: Layout redone, schematics simplified
Parts:
- removed J1, J4: CONN_02X03, OpenC16Cart:Pin_Header_Straight_2x03-ModSilkS, symbol CONN_02X03
- removed J11, J12, J2, J21, J22, J3, J5, J6: CONN_01X03, OpenC16Cart:Pin_Header_Straight_1x03-ModSilkS, symbol CONN_01X03
- removed J7: C16-Exp-Port, OpenC16Cart:C16_Cart_Conn, symbol C16-Exp-Port
- added J5: C16-Exp-Port, OpenC16Cart:C16_Cart_Conn, symbol C16-Exp-Port:C16-Exp-Port
- added JP1: U1 A14/~PGM, Jumper:SolderJumper-2_P1.3mm_Open_RoundedPad1.0x1.5mm, symbol Jumper:SolderJumper_2_Open
- added JP2: U1 A15/VPP, Jumper:SolderJumper-2_P1.3mm_Open_RoundedPad1.0x1.5mm, symbol Jumper:SolderJumper_2_Open
- added JP3: U2 A14/~PGM, Jumper:SolderJumper-2_P1.3mm_Open_RoundedPad1.0x1.5mm, symbol Jumper:SolderJumper_2_Open
- added JP4: U2 A15/VPP, Jumper:SolderJumper-2_P1.3mm_Open_RoundedPad1.0x1.5mm, symbol Jumper:SolderJumper_2_Open
- added R1, R2, R3, R4: 10kΩ, Resistor_SMD:R_0805_2012Metric_Pad1.15x1.40mm_HandSolder, symbol Device:R_Small
- added SW1: SW_DIP_x04, Button_Switch_THT:SW_DIP_SPSTx04_Piano_10.8x11.72mm_W7.62mm_P2.54mm, symbol Switch:SW_DIP_x04
- C1, C2: symbol C -> Device:C
- U1: value 27512 - LO ROM -> LO ROM; symbol 27512 -> OpenC16Cart-rescue:27512-OpenC16Cart-rescue
- U2: value 27512 - HI ROM -> HI ROM; symbol 27512 -> OpenC16Cart-rescue:27512-OpenC16Cart-rescue
Connections:
- net labels added: U1-A14, U1-A15, U2-A14, U2-A15, a11, a13
- net labels removed: /ce_u1, /ce_u2, a11_conn, a11_u1, a11_u2, a13_conn, a13_u1, a13_u2, a14_u1, a14_u2, a15_u1, a15_u2
- wire segments 132 -> 141
- no-connect marks 17 -> 20
